File: minicurso.sch (KiCad schematic (older format))
At the start: 5 parts

Commit message: Footprints selecionadas
Parts:
- gave numbers to parts that had none: 5
Changed lines of the file:
@@
 $EndDescr
 $Comp
-L Device:R_Small R?
+L Device:R_Small R1
 U 1 1 5D4DF63B
 P 4450 3750
-F 0 "R?" V 4254 3750 50  0000 C CNN
+F 0 "R1" V 4254 3750 50  0000 C CNN
 F 1 "1k" V 4345 3750 50  0000 C CNN
 F 2 "" H 4450 3750 50  0001 C CNN
@@
 $EndComp
 $Comp
-L Device:R_Small R?
+L Device:R_Small R3
 U 1 1 5D4E19C9
 P 5250 4150
-F 0 "R?" H 5191 4104 50  0000 R CNN
+F 0 "R3" H 5191 4104 50  0000 R CNN
 F 1 "10k" H 5191 4195 50  0000 R CNN
 F 2 "" H 5250 4150 50  0001 C CNN
@@
 $EndComp
 $Comp
-L Device:C_Small C?
+L Device:C_Small C1
 U 1 1 5D4E2804
 P 4100 3750
-F 0 "C?" V 3871 3750 50  0000 C CNN
+F 0 "C1" V 3871 3750 50  0000 C CNN
 F 1 "20nF" V 3962 3750 50  0000 C CNN
 F 2 "" H 4100 3750 50  0001 C CNN
@@
 $EndComp
 $Comp
-L Transistor_BJT:BC548 Q?
+L Transistor_BJT:BC548 Q1
 U 1 1 5D4E2ED4
 P 5150 3750
-F 0 "Q?" H 5341 3796 50  0000 L CNN
+F 0 "Q1" H 5341 3796 50  0000 L CNN
 F 1 "BC548" H 5341 3705 50  0000 L CNN
 F 2 "Package_TO_SOT_THT:TO-92_Inline" H 5350 3675 50  0001 L CIN
@@
 $EndComp
 $Comp
-L Device:R_Small R?
+L Device:R_Small R2
 U 1 1 5D4E360B
 P 4750 4000
-F 0 "R?" H 4691 3954 50  0000 R CNN
+F 0 "R2" H 4691 3954 50  0000 R CNN
 F 1 "510k" H 4691 4045 50  0000 R CNN
 F 2 "" H 4750 4000 50  0001 C CNN
@@
 $EndComp
 $Comp
-L power:GND #PWR?
+L power:GND #PWR0101
 U 1 1 5D4E5BAD
 P 5250 4500
-F 0 "#PWR?" H 5250 4250 50  0001 C CNN
+F 0 "#PWR0101" H 5250 4250 50  0001 C CNN
 F 1 "GND" H 5255 4327 50  0000 C CNN
 F 2 "" H 5250 4500 50  0001 C CNN
@@
 $EndComp
 $Comp
-L power:VCC #PWR?
+L power:VCC #PWR0102
 U 1 1 5D4E638A
 P 5250 3250
-F 0 "#PWR?" H 5250 3100 50  0001 C CNN
+F 0 "#PWR0102" H 5250 3100 50  0001 C CNN
 F 1 "VCC" H 5267 3423 50  0000 C CNN
 F 2 "" H 5250 3250 50  0001 C CNN
@@
 	4750 3750 4950 3750
 $Comp
-L power:GND #PWR?
+L power:GND #PWR0103
 U 1 1 5D4E819C
 P 4750 4400
-F 0 "#PWR?" H 4750 4150 50  0001 C CNN
+F 0 "#PWR0103" H 4750 4150 50  0001 C CNN
 F 1 "GND" H 4755 4227 50  0000 C CNN
 F 2 "" H 4750 4400 50  0001 C CNN

Commit message: Atualização(@
Parts:
- C1: footprint (none) -> Capacitor_THT:C_Disc_D3.0mm_W2.0mm_P2.50mm
- R1, R2, R3: footprint (none) -> Resistor_THT:R_Axial_DIN0204_L3.6mm_D1.6mm_P7.62mm_Horizontal
Changed lines of the file:
@@
 F 0 "R1" V 4254 3750 50  0000 C CNN
 F 1 "1k" V 4345 3750 50  0000 C CNN
-F 2 "" H 4450 3750 50  0001 C CNN
+F 2 "Resistor_THT:R_Axial_DIN0204_L3.6mm_D1.6mm_P7.62mm_Horizontal" H 4450 3750 50  0001 C CNN
 F 3 "~" H 4450 3750 50  0001 C CNN
 	1    4450 3750
@@
 F 0 "R3" H 5191 4104 50  0000 R CNN
 F 1 "10k" H 5191 4195 50  0000 R CNN
-F 2 "" H 5250 4150 50  0001 C CNN
+F 2 "Resistor_THT:R_Axial_DIN0204_L3.6mm_D1.6mm_P7.62mm_Horizontal" H 5250 4150 50  0001 C CNN
 F 3 "~" H 5250 4150 50  0001 C CNN
 	1    5250 4150
@@
 F 0 "C1" V 3871 3750 50  0000 C CNN
 F 1 "20nF" V 3962 3750 50  0000 C CNN
-F 2 "" H 4100 3750 50  0001 C CNN
+F 2 "Capacitor_THT:C_Disc_D3.0mm_W2.0mm_P2.50mm" H 4100 3750 50  0001 C CNN
 F 3 "~" H 4100 3750 50  0001 C CNN
 	1    4100 3750
@@
 F 0 "R2" H 4691 3954 50  0000 R CNN
 F 1 "510k" H 4691 4045 50  0000 R CNN
-F 2 "" H 4750 4000 50  0001 C CNN
+F 2 "Resistor_THT:R_Axial_DIN0204_L3.6mm_D1.6mm_P7.62mm_Horizontal" H 4750 4000 50  0001 C CNN
 F 3 "~" H 4750 4000 50  0001 C CNN
 	1    4750 4000
